Commit message: Add files via upload

File: src/demo_arm_description/urdf/project.urdf.xacro (robot description, xacro)
@@ -209,4 +209,13 @@
         <mimic joint="joint_4" multiplier="-1"/>
     </joint>
+    <!-- <joint name ="joint_5_mimic" type="revolute">
+        <parent link="claw_support"/>
+        <child link = "gripper_left"/>
+        <origin xyz="-0.22 0.13 -0.1"/>
+        <axis xyz="0 0 1"/>
+        <limit lower="0.0" upper="${PI/2}"
+            effort="${effort}" velocity="${velocity}"/>
+        <mimic joint="joint_4" multiplier="-1"/>
+    </joint> -->
     <!-- <Adding colour to arm in Gazebo> -->
     <gazebo reference="base_link">
